File: sx1255_eval.kicad_sch (KiCad schematic)
At the start: 26 parts, among them IC1 SX1255, J1 EXT_CLK_IN, J2 TX_SMA, J3 RX_SMA, J4 CONN

Commit message: WIP PCB layout
Parts:
- C1, C2: LCSC Part# (none) -> C100042
- C10, C3, C4, C5, C6, C7: LCSC Part# (none) -> C14663
- C8: LCSC Part# (none) -> C107047
- C9: LCSC Part# (none) -> C107045
- IC1: LCSC Part# (none) -> C89372
- J1: footprint Connector_Coaxial:U.FL_Molex_MCRF_73412-0110_Vertical -> Connector_Coaxial:U.FL_Hirose_U.FL-R-SMT-1_Vertical; LCSC Part# (none) -> C434812
- J2, J3: LCSC Part# (none) -> -
- J4: LCSC Part# (none) -> C2884018
- L1: LCSC Part# (none) -> C346329
- L2: LCSC Part# (none) -> C74308
- R1, R2, R3, R4, R5, R6, R7, R8, R9: LCSC Part# (none) -> C125923
Changed lines of the file:
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@@
   (title_block
     (title "SX1255 Evaluation Board")
-    (date "17.12.2023")
+    (date "18.12.2023")
     (rev "A")
     (company "Wojciech Kaczmarski SP5WWP, M17 Project")
@@
       (effects (font (size 1.27 1.27)) hide)
     )
+    (property "LCSC Part#" "C14663" (at 107.95 104.14 0)
+      (effects (font (size 1.27 1.27)) hide)
+    )
     (pin "1")
     (pin "2")
@@
     )
     (property "MPN" "C0603C104M5RAC7411" (at 81.28 132.08 0)
+      (effects (font (size 1.27 1.27)) hide)
+    )
+    (property "LCSC Part#" "C14663" (at 81.28 132.08 0)
       (effects (font (size 1.27 1.27)) hide)
     )
@@
       (effects (font (size 1.27 1.27)) hide)
     )
+    (property "LCSC Part#" "-" (at 129.54 54.61 0)
+      (effects (font (size 1.27 1.27)) hide)
+    )
     (pin "1")
     (pin "2")
@@
     )
     (property "MPN" "C0603C104M5RAC7411" (at 116.84 104.14 0)
+      (effects (font (size 1.27 1.27)) hide)
+    )
+    (property "LCSC Part#" "C14663" (at 116.84 104.14 0)
       (effects (font (size 1.27 1.27)) hide)
     )
@@
       (effects (font (size 1.27 1.27)) hide)
     )
+    (property "LCSC Part#" "C100042" (at 54.61 132.08 0)
+      (effects (font (size 1.27 1.27)) hide)
+    )
     (pin "1")
     (pin "2")
@@
     )
     (property "MPN" "C0603C104M5RAC7411" (at 99.06 104.14 0)
+      (effects (font (size 1.27 1.27)) hide)
+    )
+    (property "LCSC Part#" "C14663" (at 99.06 104.14 0)
       (effects (font (size 1.27 1.27)) hide)
     )
@@
       (effects (font (size 1.27 1.27)) hide)
     )
+    (property "LCSC Part#" "C125923" (at 143.51 135.89 0)
+      (effects (font (size 1.27 1.27)) hide)
+    )
     (pin "1")
     (pin "2")
@@
       (effects (font (size 1.27 1.27)) hide)
     )
+    (property "LCSC Part#" "C125923" (at 173.99 102.87 0)
+      (effects (font (size 1.27 1.27)) hide)
+    )
     (pin "1")
     (pin "2")
@@
     )
     (property "MPN" "538-15-91-2180" (at 222.25 97.79 0)
+      (effects (font (size 1.27 1.27)) hide)
+    )
+    (property "LCSC Part#" "C2884018" (at 222.25 97.79 0)
       (effects (font (size 1.27 1.27)) hide)
     )
@@
       (effects (font (size 1.27 1.27)) hide)
     )
+    (property "LCSC Part#" "C107047" (at 138.43 54.61 0)
+      (effects (font (size 1.27 1.27)) hide)
+    )
     (pin "1")
     (pin "2")
@@
       (effects (font (size 1.27 1.27)) hide)
     )
+    (property "LCSC Part#" "C125923" (at 148.59 135.89 0)
+      (effects (font (size 1.27 1.27)) hide)
+    )
     (pin "1")
     (pin "2")
@@
       (effects (font (size 1.27 1.27)) hide)
     )
+    (property "LCSC Part#" "C125923" (at 153.67 135.89 0)
+      (effects (font (size 1.27 1.27)) hide)
+    )
     (pin "1")
     (pin "2")
@@
       (effects (font (size 1.27 1.27)) hide)
     )
+    (property "LCSC Part#" "C346329" (at 162.56 49.53 0)
+      (effects (font (size 1.27 1.27)) hide)
+    )
     (pin "1")
     (pin "2")
@@
       (effects (font (size 1.27 1.27)) hide)
     )
+    (property "LCSC Part#" "C125923" (at 146.05 135.89 0)
+      (effects (font (size 1.27 1.27)) hide)
+    )
     (pin "1")
     (pin "2")
@@
       (effects (font (size 1.27 1.27)) hide)
     )
+    (property "LCSC Part#" "C107045" (at 146.05 44.45 0)
+      (effects (font (size 1.27 1.27)) hide)
+    )
     (pin "1")
     (pin "2")
@@
       (effects (font (size 1.27 1.27)) hide)
     )
+    (property "LCSC Part#" "C125923" (at 173.99 105.41 0)
+      (effects (font (size 1.27 1.27)) hide)
+    )
     (pin "1")
     (pin "2")
@@
       (effects (font (size 1.27 1.27)) hide)
     )
+    (property "LCSC Part#" "C14663" (at 172.72 72.39 0)
+      (effects (font (size 1.27 1.27)) hide)
+    )
     (pin "1")
     (pin "2")
@@
     )
     (property "MPN" "-" (at 177.8 44.45 0)
+      (effects (font (size 1.27 1.27)) hide)
+    )
+    (property "LCSC Part#" "-" (at 177.8 44.45 0)
       (effects (font (size 1.27 1.27)) hide)
     )
@@
     )
     (property "MPN" "CRCW0603100RFKECC" (at 173.99 107.95 0)
+      (effects (font (size 1.27 1.27)) hide)
+    )
+    (property "LCSC Part#" "C125923" (at 173.99 107.95 0)
       (effects (font (size 1.27 1.27)) hide)
     )
@@
       (effects (font (size 1.27 1.27)) hide)
     )
+    (property "LCSC Part#" "C100042" (at 63.5 132.08 0)
+      (effects (font (size 1.27 1.27)) hide)
+    )
     (pin "1")
     (pin "2")
@@
       (effects (font (size 1.27 1.27)) (justify left))
     )
-    (property "Footprint" "Connector_Coaxial:U.FL_Molex_MCRF_73412-0110_Vertical" (at 67.31 95.25 0)
+    (property "Footprint" "Connector_Coaxial:U.FL_Hirose_U.FL-R-SMT-1_Vertical" (at 67.31 95.25 0)
       (effects (font (size 1.27 1.27)) hide)
     )
@@
     )
     (property "MPN" "CONUFL001-SMD-T" (at 67.31 95.25 0)
+      (effects (font (size 1.27 1.27)) hide)
+    )
+    (property "LCSC Part#" "C434812" (at 67.31 95.25 0)
       (effects (font (size 1.27 1.27)) hide)
     )
@@
       (effects (font (size 1.27 1.27)) hide)
     )
+    (property "LCSC Part#" "C125923" (at 156.21 135.89 0)
+      (effects (font (size 1.27 1.27)) hide)
+    )
     (pin "1")
     (pin "2")
@@
     )
     (property "PN" "947-SX1255IWLTRT" (at 133.35 90.17 0)
+      (effects (font (size 1.27 1.27)) hide)
+    )
+    (property "LCSC Part#" "C89372" (at 133.35 90.17 0)
       (effects (font (size 1.27 1.27)) hide)
     )
@@
       (effects (font (size 1.27 1.27)) hide)
     )
+    (property "LCSC Part#" "C125923" (at 151.13 135.89 0)
+      (effects (font (size 1.27 1.27)) hide)
+    )
     (pin "1")
     (pin "2")
@@
       (effects (font (size 1.27 1.27)) hide)
     )
+    (property "LCSC Part#" "C74308" (at 167.64 44.45 0)
+      (effects (font (size 1.27 1.27)) hide)
+    )
     (pin "1")
     (pin "2")
@@
       (effects (font (size 1.27 1.27)) hide)
     )
+    (property "LCSC Part#" "C14663" (at 72.39 132.08 0)
+      (effects (font (size 1.27 1.27)) hide)
+    )

Commit message: WIP PCB
Parts:
- added C1: 10n, Capacitor_SMD:C_0603_1608Metric, symbol Device:C_Small
- added C6: 100n, Capacitor_SMD:C_0603_1608Metric, symbol Device:C_Small
- renumbered C8 to C10, C9 to C11, C10 to C12, C1 to C2, C2 to C3, C3 to C4, C4 to C5, C5 to C7, C6 to C8, C7 to C9
Connections:
- net +3V3: now also C1.1, C6.1
- net GND: now also C1.2, C6.2
Other:
- moved on the sheet: C2, C3, C4, C5

Commit message: PMOD
Parts:
- removed J4: CONN, Connector_PinHeader_2.54mm:PinHeader_2x09_P2.54mm_Vertical_SMD, symbol Connector_Generic:Conn_02x09_Odd_Even
- added J4, J5: PMOD, Connector_PinHeader_2.54mm:PinHeader_2x06_P2.54mm_Horizontal, symbol Connector_Generic:Conn_02x06_Odd_Even
- added JP1: EXT_CLK_SRC, Connector_PinHeader_2.54mm:PinHeader_1x03_P2.54mm_Vertical, symbol Jumper:Jumper_3_Bridged12
- J1: footprint Connector_Coaxial:U.FL_Hirose_U.FL-R-SMT-1_Vertical -> Connector_Coaxial:SMA_Samtec_SMA-J-P-X-ST-EM1_EdgeMount; LCSC Part# C434812 -> -; MPN CONUFL001-SMD-T -> -; PN CONUFL001-SMD-T -> -
- renumbered C7 to C6, C6 to C7
Connections:
- net +3V3: now also J4.1 (Pin_1), J4.2 (Pin_2), J5.1 (Pin_1), J5.2 (Pin_2)
- net CK_IN: now also J5.9 (Pin_9)
- net CK_OUT: now also J5.10 (Pin_10)
- net DIO0: now also J4.8 (Pin_8)
- net DIO1: now also J4.7 (Pin_7)
- net DIO2: now also J4.6 (Pin_6)
- net DIO3: now also J4.5 (Pin_5)
- net EXT_CLK: now also JP1.2 (C); no longer J1.1 (In)
- net GND: now also J4.3 (Pin_3), J4.4 (Pin_4), J5.3 (Pin_3), J5.4 (Pin_4)
- net I_IN: now also J5.7 (Pin_7)
- net I_OUT: now also J5.5 (Pin_5)
- net MISO: now also J4.10 (Pin_10)
- net MOSI: now also J4.11 (Pin_11)
- net Q_IN: now also J5.8 (Pin_8)
- net Q_OUT: now also J5.6 (Pin_6)
- net RST: now also J5.11 (Pin_11)
- net SCK: now also J4.12 (Pin_12)
- net ~{CS}: now also J4.9 (Pin_9)
- net RF_OUT: now reaches C10.2, J2.1 (In)
- net RF_IN: now reaches J3.1 (In), L2.1
- new net EXT_CLK_A: J5.12 (Pin_12), JP1.3 (B)
- new net EXT_CLK_B: J1.1 (In), JP1.1 (A)
Other:
- moved on the sheet: J1, J2, J3

Commit message: PN update, gerbers
minor silkscreen tweaks
Parts:
- J1, J2, J3: LCSC Part# - -> C2913580
- J4, J5: LCSC Part# (none) -> C706886
- JP1: LCSC Part# (none) -> C6332196
Changed lines of the file:
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@@
       (effects (font (size 1.27 1.27)) hide)
     )
-    (property "LCSC Part#" "" (at 224.79 68.58 0)
+    (property "LCSC Part#" "C706886" (at 224.79 68.58 0)
       (effects (font (size 1.27 1.27)) hide)
     )
@@
       (effects (font (size 1.27 1.27)) hide)
     )
-    (property "LCSC Part#" "-" (at 123.19 54.61 0)
+    (property "LCSC Part#" "C2913580" (at 123.19 54.61 0)
       (effects (font (size 1.27 1.27)) hide)
     )
@@
       (effects (font (size 1.27 1.27)) hide)
     )
-    (property "LCSC Part#" "" (at 224.79 109.22 0)
+    (property "LCSC Part#" "C706886" (at 224.79 109.22 0)
       (effects (font (size 1.27 1.27)) hide)
     )
@@
       (effects (font (size 1.27 1.27)) hide)
     )
-    (property "LCSC Part#" "-" (at 181.61 44.45 0)
+    (property "LCSC Part#" "C2913580" (at 181.61 44.45 0)
       (effects (font (size 1.27 1.27)) hide)
     )
@@
       (effects (font (size 1.27 1.27)) hide)
     )
-    (property "LCSC Part#" "-" (at 91.44 44.45 0)
+    (property "LCSC Part#" "C2913580" (at 91.44 44.45 0)
       (effects (font (size 1.27 1.27)) hide)
     )
@@
       (effects (font (size 1.27 1.27)) hide)
     )
-    (property "LCSC Part#" "" (at 88.9 68.58 0)
-      (effects (font (size 1.27 1.27)) hide)
-    )
+    (property "LCSC Part#" "C6332196" (at 88.9 68.58 0)
+      (effects (font (size 1.27 1.27)) hide)
+    )

Commit message: BOM update
J4, J5 had wrong PN assigned (2x05 instead of 2x06 headers)
Parts:
- J4, J5: LCSC Part# C706886 -> C706887
Changed lines of the file:
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@@
       (effects (font (size 1.27 1.27)) hide)
     )
-    (property "LCSC Part#" "C706886" (at 224.79 68.58 0)
+    (property "LCSC Part#" "C706887" (at 224.79 68.58 0)
       (effects (font (size 1.27 1.27)) hide)
     )
@@
       (effects (font (size 1.27 1.27)) hide)
     )
-    (property "LCSC Part#" "C706886" (at 224.79 109.22 0)
-      (effects (font (size 1.27 1.27)) hide)
-    )
+    (property "LCSC Part#" "C706887" (at 224.79 109.22 0)
+      (effects (font (size 1.27 1.27)) hide)
+    )

Commit message: updated SMA conn PN
removed fab files
Parts:
- J1, J2, J3: LCSC Part# C2913580 -> C496550
Changed lines of the file:
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@@
       (effects (font (size 1.27 1.27)) hide)
     )
-    (property "LCSC Part#" "C2913580" (at 123.19 54.61 0)
+    (property "LCSC Part#" "C496550" (at 123.19 54.61 0)
       (effects (font (size 1.27 1.27)) hide)
     )
@@
       (effects (font (size 1.27 1.27)) hide)
     )
-    (property "LCSC Part#" "C2913580" (at 181.61 44.45 0)
+    (property "LCSC Part#" "C496550" (at 181.61 44.45 0)
       (effects (font (size 1.27 1.27)) hide)
     )
@@
       (effects (font (size 1.27 1.27)) hide)
     )
-    (property "LCSC Part#" "C2913580" (at 91.44 44.45 0)
-      (effects (font (size 1.27 1.27)) hide)
-    )
+    (property "LCSC Part#" "C496550" (at 91.44 44.45 0)
+      (effects (font (size 1.27 1.27)) hide)
+    )
